File: MAKEEN_Keypad_Test_PCB.kicad_pcb (KiCad board)
At the start: 2 copper layers, 56 x 65 mm, 20 parts, among them J1 Keypad_Conn, J2 Pi5_Conn_GPIO, J3 3V3_IN_Conn

Commit message: Routing
Routing:
- net KB_IN_ROW4: track 22.3 -> 92.0 mm, vias 2 -> 4
- net KB_IN_ROW1: track 37.1 -> 106.5 mm, vias 1 -> 3
- net  KB_IN_ROW2: track 27.5 -> 95.9 mm, vias 2 -> 4
- net KB_IN_ROW3: track 33.3 -> 100.3 mm, vias 2 -> 4
- net KB_IN_ROW5: track 30.9 -> 96.2 mm, vias 2 -> 3
- net KB_OUT_COL1: track 12.7 -> 45.9 mm, vias 0 -> 1
- net KB_OUT_COL4: track 11.3 -> 42.1 mm, vias 0 -> 2
- net KB_OUT_COL2: track 9.00 -> 39.1 mm, vias 0 -> 3
- net KB_OUT_COL3: track 14.6 -> 42.0 mm, vias 0 -> 2
Other:
- outline, holes or cut-outs redrawn

Commit message: V1-completed
Parts:
- added G***: LOGO, MAKEEN_Keypad_Test_PCB:GPV_logo_20mm, F.Cu at (145.7, 88.0)
Routing:
- net KB_OUT_COL3: track 42.0 -> 43.9 mm
- net KB_OUT_COL4: track 42.1 -> 43.6 mm
- net KB_IN_ROW3: track 100.3 -> 101.0 mm
- net  KB_IN_ROW2: track 95.9 -> 96.6 mm
- net KB_IN_ROW1: track 106.5 -> 105.9 mm
Other:
- board text added: "KB_IN_ROW Resistors"
- board text added: "KB_OUT_COL Resistors"
- board text added: "MAKEEN - Keypad Tester PCB Rpi HAT - XS01A00003638F V1-25.0815 ©ls"
- board text added: "Pull Down"
- board text added: "Pull Up"
